File: electric/digirig-light.kicad_sch (KiCad schematic)
At the start: 22 parts, among them J1 USB_A, J2 PJ-320A, Q1 MMBT5551L, U1 CM108B

Commit message: Revision 1.1
- PTT by tone circuit modification
- CM108B output voltage config change from 2.5V to 3.5V
Parts:
- added C4: 1uF, Capacitor_SMD:C_0402_1005Metric, symbol Device:C
- added D1: GS2005ELD, Diode_SMD:D_SOD-923, symbol Device:D_Schottky
- added R6: 1K5, Resistor_SMD:R_0402_1005Metric, symbol Device:R_US
- C6: renamed from C7; value 100n -> 1uF; LCSC C1525 -> C52923
- renumbered C9 to C10, C4 to C5, C5 to C7, C6 to C8, C8 to C9, D1 to D2, R3 to R2, R2 to R3, R6 to R7, R7 to R8
Connections:
- net +5V: now also U1.28 (VSEL)
- net GND: now also D1.2 (A); no longer U1.28 (VSEL)
- net ROUT: now also R3.1; no longer D2.2 (A)
- net at C6.1, R2.1, R5.2: now also D2.1 (K), R6.2; no longer Q1.1 (B), R3.2
- new net: Q1.1 (B), R6.1
- new net: C4.1, D1.1 (K), D2.2 (A)
- new net: C4.2, R3.2
Other:
- note added: "CM108 Config: - Playback & Recording (MODE low) - With Mixer / AA-Path Enable (MSEL high) - Line out Vpp = 3.5 Volts (VSEL high) - Bus Power with 100mA (PWRSEL high) - Use internal ADC (ADSEL low) - Normal Operation (TEST low)"
- note removed: "CM108 Config: - Playback & Recording (MODE low) - With Mixer / AA-Path Enable (MSEL high) - Line out Vpp = 2.5 Volts (VSEL low) - Bus Power with 100mA (PWRSEL high) - Use internal ADC (ADSEL low) - Normal Operation (TEST low)"
- moved on the sheet: C6, D2, R2, R3, R5
