File: electric/digirig-lite.kicad_sch (KiCad schematic)
At the start: 54 parts, among them Q1 MMBT5551L, Q2 MMBT5551L, Q3 MMBT5551L, U1 CM108

Commit message: Revision 1.2
Parts:
- Q1, Q2, Q3: LCSC C152516 -> C2145
- TP10, TP5: now left out of the parts list
